File: Hardware/ARTIC_R2_Module.sch (EAGLE design)
At the start: 94 parts, among them J1 U.FL, K1 TLP3475R, Q2 5.8A/30V/35mΩ, U1 ADM4210-1, U2 1.8V/100mA, U3 ARTIC_R2, U4 RFPA0133, U5 AS179-92LF, U6 3.0V, X1 CRYSTAL-TCXO-26MHZ

Commit message: Work in progress
Parts:
- added J10, J11, J12, J13, J14, J15, J16, J17, J18, J19, J2, J20, J21, J22, J23, J24, J3, J4, J5, J6, J7, J8, J9: (no value), SparkFun-Connectors:CONN_01PTH_NO_SILK_YES_STOP
- added J25: U.FL, SparkFun-Connectors:U.FL2PIN
- J1: value U.FL -> (none); device SparkFun-Connectors:U.FL2PIN -> SparkFun-Connectors:CONN_01PTH_NO_SILK_YES_STOP
Connections:
- net ANTENNA: now also J23.1, J25.SIGNAL; no longer J1.SIGNAL
- net FLSH_CEN: now also J20.1
- net FLSH_SCLK: now also J17.1
- net FLSH_SI: now also J18.1
- net FLSH_SO: now also J19.1
- net GND: now also J16.1, J22.1, J24.1, J25.GND; no longer J1.GND
- net PWR_EN: now also J13.1
- net VDD: now also J21.1
- net VIN: now also J14.1, J15.1
Other:
- note added: "Pads"
- note removed: "Pins"
- moved on the sheet: K1

Commit message: Adding panel files. Updating README.
Parts:
- removed LOGO3: OSHW-LOGOS, SparkFun-Aesthetics:OSHW-LOGOS
- removed SPARKX1, SPARKX2: SPARKX-LOGO4, SparkX:SPARKX-LOGO4
- added SCREEN: ARTIC_R2_CASTELLATED_CAN, New_Parts_Screening_Cans:ARTIC_R2_CASTELLATED_CAN
- J1, J10, J11, J12, J13, J14, J15, J16, J17, J18, J19, J2, J20, J21, J22, J23, J24, J3, J4, J5, J6, J7, J8, J9: device SparkFun-Connectors:CONN_01PTH_NO_SILK_YES_STOP -> New_Parts_Connectors:CONN_01_CASTELLATEDCASTELLATED
- R9: value 0.012R -> 0.1R; device New_Parts:RESISTOR_0603_12MILLIOHM0603 -> New_Parts_Resistors:RESISTOR_0603_100MILLIOHM0603
- U1: device New_Parts:ADM4210-1 -> New_Parts_IC-Power:ADM4210-1
Connections:
- net 1.8V: now also J11.1
- net BOOT: now also J3.1
- net CIPO: now also J10.1
- net COPI: now also J9.1
- net CS: now also J7.1
- net G8: now also J1.1
- net GND: now also J12.1, SCREEN.P$1
- net INT1: now also J4.1
- net INT2: now also J5.1
- net RESETB: now also J6.1
- net SCLK: now also J8.1
- net VREF1: now also J2.1
Other:
- note added: "Current Limit: 500mA ADM4210-1 VCB: 50mV Sense Resistor: 0.1 Ohms"
- note added: "Pads & Can"
- note removed: "Pads"
- moved on the sheet: C1, C2, C23, C30, C31, C36, C37, C42, C45, C48, C49, J25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
