File: Hardware/ARTIC_R2_Module.sch (EAGLE design)
At the start: 120 parts, among them J1 CONN_01_CASTELLATED_4LAYERWIT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, J10 CONN_01_CASTELLATED_4LAYERWIT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, J11 CONN_01_CASTELLATED_4LAYERWIT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, J12 CONN_01_CASTELLATED_4LAYERWIT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, J13 CONN_01_CASTELLATED_4LAYERWIT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, J14 CONN_01_CASTELLATED_4LAYERWIT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, J15 CONN_01_CASTELLATED_4LAYERWIT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, J16 CONN_01_CASTELLATED_4LAYERWIT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, J17 CONN_01_CASTELLATED_4LAYERWIT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, J18 CONN_01_CASTELLATED_4LAYERWIT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, J19 CONN_01_CASTELLATED_4LAYERWIT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, J2 CONN_01_CASTELLATED_4LAYERWIT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, J20 CONN_01_CASTELLATED_4LAYERWIT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, J21 CONN_01_CASTELLATED_4LAYERWIT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, J22 CONN_01_CASTELLATED_4LAYERWIT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, J23 CONN_01_CASTELLATED_4LAYERWIT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, J24 CONN_01_CASTELLATED_4LAYERWIT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, J25 U.FL, J3 CONN_01_CASTELLATED_4LAYERWIT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, J4 CONN_01_CASTELLATED_4LAYERWIT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, J5 CONN_01_CASTELLATED_4LAYERWIT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, J6 CONN_01_CASTELLATED_4LAYERWIT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, J7 CONN_01_CASTELLATED_4LAYERWIT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, J8 CONN_01_CASTELLATED_4LAYERWIT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, J9 CONN_01_CASTELLATED_4LAYERWIT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, K1 TLP3475R, Q2 5.8A/30V/35mΩ, U1 ADM4210-1, U2 1.8V/100mA, U3 ARTIC_R2, U4 RFPA0133, U5 AS179-92LF, U6 3.0V, U7 SST25VF020BUSON, X1 CRYSTAL-TCXO-26MHZ

Commit message: Update Eagle files - remove New_Parts libraries
Parts:
- C28: device New_Parts_Capacitors:9.1PF-0402-TIGHT -> SparkFun-Capacitors:9.1PF-0402-TIGHT
- J25: device SparkFun-Connectors:U.FL2PIN -> SparkFun-Connectors:U.FL2PIN-REDUCED-FOOTPRINT
- K1: device New_Parts_DiscreteSemi:TLP3475R -> SparkFun-DiscreteSemi:TLP3475R
- L11: device New_Parts_Coils:30NH-0402 -> SparkFun-Coils:30NH-0402
- L12: device New_Parts_Coils:51NH-0402 -> SparkFun-Coils:51NH-0402
- L5: device New_Parts_Coils:15NH-0402 -> SparkFun-Coils:15NH-0402
- L6: device New_Parts_Coils:27NH-0402 -> SparkFun-Coils:27NH-0402
- L7: device New_Parts_Coils:18NH-0402 -> SparkFun-Coils:18NH-0402
- L8: device New_Parts_Coils:12NH-0402 -> SparkFun-Coils:12NH-0402
- R11, R2: value 100OHM -> 100; device New_Parts_Resistors:100OHM -> SparkFun-Resistors:100OHM-0402-TIGHT-1/16W-1%
- R14: device New_Parts_Resistors:470OHM-0402-TIGHT-1/16W-1% -> SparkFun-Resistors:470OHM-0402-TIGHT-1/16W-1%
- R17: device New_Parts_Resistors:47OHM-0402-TIGHT-1/16W-1% -> SparkFun-Resistors:47OHM-0402-TIGHT-1/16W-1%
- R3: value 3.9OHM -> 3.9; device New_Parts_Resistors:3.9OHM -> SparkFun-Resistors:3.9OHM-0402-TIGHT-1/16W-1%
- R6: value 220OHM -> 220; device New_Parts_Resistors:220OHM -> SparkFun-Resistors:220OHM-0402-TIGHT-1/16W-1%
- R9: value 0.1R -> 0.1; device New_Parts_Resistors:RESISTOR_0603_100MILLIOHM0603 -> SparkFun-Resistors:0.1OHM-0603-1/3W-1%
- SCREEN: value ARTIC_R2_CASTELLATED_CAN -> IOTA_SCREENING_CANSTRAIGHT_SLOTS; device New_Parts_Screening_Cans:ARTIC_R2_CASTELLATED_CAN -> New_Parts_Screening_Cans:IOTA_SCREENING_CANSTRAIGHT_SLOTS
- U1: value ADM4210-1 -> ADM4210_1TSOT6; device New_Parts_IC-Power:ADM4210-1 -> SparkFun-IC-Power:ADM4210_1TSOT6
- U3: device New_Parts_IC-Comms:ARTIC_R2 -> SparkFun-RF:ARTIC_R2
- U4: device New_Parts_IC-Comms:RFPA0133 -> SparkFun-RF:RFPA0133
- U5: device New_Parts_IC-Comms:AS179-92LF -> SparkFun-RF:AS179-92LF
- U6: device New_Parts_IC-Power:V_REG_LP5907SOT23-3.0V -> SparkFun-IC-Power:V_REG_LP5907SOT23-3.0V
- U7: device New_Parts_IC-Memory:SST25VF020BUSON -> SparkFun-IC-Memory:SST25VF020BUSON
- X1: device New_Parts_Clocks:CRYSTAL-TCXO-26MHZ -> SparkFun-Clocks:CRYSTAL-TCXO-26MHZ
